File: Nucleo Pepi board/schematic.brd (EAGLE design)
At the start: 64.8 x 57.1 mm, 9 parts, among them J1 1X2-3.5MM

Commit message: update
Parts:
- added SJ2, SJ3: (no value), jumper:SJW
Connections:
- removed net 5V: A1.4.4
- new net N$1: A1.4.1, SJ2.1
- new net N$2: A1.4.4, SJ3.1
- net GND: no longer U$1.EN
- net VBAT: now also SJ2.2
- net VCC: now also SJ3.2
Routing:
- net VBAT: track 6.39 -> 26.8 mm
- net N$2: track 0.00 -> 13.2 mm
- net GND: track 175.4 -> 169.6 mm
- net N$1: track 0.00 -> 5.08 mm
- net VCC: track 103.1 -> 107.0 mm, vias 0 -> 1
- net PA2: track 39.9 -> 38.2 mm
- net PB3: track 34.3 -> 35.6 mm
- net PA8: track 20.0 -> 18.9 mm
Other:
- board size 64.8 x 57.1 mm -> 64.8 x 67.3 mm
- board text added: "PB4"
- board text added: "Pepi Board Ver 1.2"
- board text added: "_"
- board text removed: "-"
- board text removed: "Pepi Board Ver 1"

Commit message: maj
Parts:
- removed SJ2: (no value), jumper:SJW
- added VBAT: (no value), jumper:SJW
- renumbered SJ3 to 5V
Connections:
- net N$1: now also VBAT.1; no longer SJ2.1
- net VBAT: now also VBAT.2; no longer SJ2.2
Routing:
- net VBAT: track 26.8 -> 27.3 mm
- net N$1: track 5.08 -> 5.61 mm
Other:
- outline, holes or cut-outs redrawn
Changed lines of the file:
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@@
 <?xml version="1.0" encoding="utf-8"?>
 <!DOCTYPE eagle SYSTEM "eagle.dtd">
-<eagle version="9.3.0">
+<eagle version="9.4.2">
 <drawing>
 <settings>
@@
 <setting verticaltext="up"/>
 </settings>
-<grid distance="25" unitdist="mil" unit="mil" style="dots" multiple="1" display="yes" altdistance="5" altunitdist="mil" altunit="mil"/>
+<grid distance="50" unitdist="mil" unit="mil" style="dots" multiple="1" display="yes" altdistance="5" altunitdist="mil" altunit="mil"/>
 <layers>
 <layer number="1" name="Top" color="4" fill="1" visible="yes" active="yes"/>
@@
 <layer number="23" name="tOrigins" color="15" fill="1" visible="yes" active="yes"/>
 <layer number="24" name="bOrigins" color="15" fill="1" visible="yes" active="yes"/>
-<layer number="25" name="tNames" color="7" fill="1" visible="yes" active="yes"/>
+<layer number="25" name="tNames" color="7" fill="1" visible="no" active="yes"/>
 <layer number="26" name="bNames" color="7" fill="1" visible="yes" active="yes"/>
-<layer number="27" name="tValues" color="7" fill="1" visible="yes" active="yes"/>
+<layer number="27" name="tValues" color="7" fill="1" visible="no" active="yes"/>
 <layer number="28" name="bValues" color="7" fill="1" visible="yes" active="yes"/>
 <layer number="29" name="tStop" color="7" fill="3" visible="yes" active="yes"/>
@@
 <wire x1="25.4" y1="53.34" x2="26.67" y2="54.61" width="0.1524" layer="20"/>
 <hole x="24.13" y="57.785" drill="3.048"/>
-<wire x1="19.685" y1="52.07" x2="19.685" y2="53.34" width="0.1524" layer="20"/>
-<wire x1="19.685" y1="53.34" x2="25.4" y2="53.34" width="0.1524" layer="20"/>
 <wire x1="0" y1="53.34" x2="17.145" y2="53.34" width="0.1524" layer="20"/>
 <wire x1="17.145" y1="53.34" x2="17.145" y2="52.07" width="0.1524" layer="20"/>
 <wire x1="17.145" y1="52.07" x2="-1.27" y2="52.07" width="0.1524" layer="20"/>
-<wire x1="19.685" y1="52.07" x2="39.37" y2="52.07" width="0.1524" layer="20"/>
-<wire x1="41.91" y1="52.07" x2="58.42" y2="52.07" width="0.1524" layer="20"/>
-<wire x1="39.37" y1="52.07" x2="41.91" y2="52.07" width="0.1524" layer="20"/>
+<wire x1="25.4" y1="53.34" x2="19.05" y2="53.34" width="0.1524" layer="20"/>
+<wire x1="19.05" y1="53.34" x2="19.05" y2="52.07" width="0.1524" layer="20"/>
+<wire x1="19.05" y1="52.07" x2="58.42" y2="52.07" width="0.1524" layer="20"/>
 </plain>
 <attributes>
@@
 <attribute name="VALUE" x="31.75" y="40.005" size="0.4064" layer="27" ratio="10"/>
 </element>
-<element name="SERVO1" library="lib2" package="HEADER3X5" value="HEADER3X5" x="17.78" y="1.27" smashed="yes" rot="R180">
+<element name="SERVO1" library="lib2" package="HEADER3X5" value="HEADER3X5" x="17.78" y="1.27" locked="yes" smashed="yes" rot="R180">
 <attribute name="NAME" x="22.86" y="-3.175" size="0.8128" layer="25" ratio="18" rot="R180"/>
 </element>
@@
 <attribute name="VALUE" x="26.035" y="49.53" size="1.27" layer="27" rot="R270"/>
 </element>
-<element name="SJ2" library="jumper" library_urn="urn:adsk.eagle:library:252" package="SJW" package3d_urn="urn:adsk.eagle:package:15507/1" value="" x="7.62" y="22.86" smashed="yes" rot="MR0">
-<attribute name="NAME" x="9.779" y="24.638" size="1.27" layer="26" ratio="10" rot="MR0"/>
-<attribute name="VALUE" x="6.62" y="22.86" size="0.02" layer="28" rot="MR0"/>
+<element name="VBAT" library="jumper" library_urn="urn:adsk.eagle:library:252" package="SJW" package3d_urn="urn:adsk.eagle:package:15507/1" value="" x="8.89" y="22.86" smashed="yes" rot="MR0">
+<attribute name="NAME" x="11.049" y="24.638" size="1.27" layer="26" ratio="10" rot="MR0"/>
+<attribute name="VALUE" x="7.89" y="22.86" size="0.02" layer="28" rot="MR0"/>
 </element>
-<element name="SJ3" library="jumper" library_urn="urn:adsk.eagle:library:252" package="SJW" package3d_urn="urn:adsk.eagle:package:15507/1" value="" x="8.89" y="17.78" smashed="yes" rot="MR0">
+<element name="5V" library="jumper" library_urn="urn:adsk.eagle:library:252" package="SJW" package3d_urn="urn:adsk.eagle:package:15507/1" value="" x="8.89" y="17.78" smashed="yes" rot="MR0">
 <attribute name="NAME" x="11.049" y="19.558" size="1.27" layer="26" ratio="10" rot="MR0"/>
 <attribute name="VALUE" x="7.89" y="17.78" size="0.02" layer="28" rot="MR0"/>
@@
 <wire x1="7.62" y1="33.655" x2="22.225" y2="48.26" width="1.27" layer="1"/>
 <wire x1="22.225" y1="48.26" x2="29.21" y2="48.26" width="1.27" layer="1"/>
-<contactref element="SJ3" pad="2"/>
+<contactref element="5V" pad="2"/>
 <wire x1="7.62" y1="17.78" x2="7.591590625" y2="17.808409375" width="0.762" layer="16"/>
 <wire x1="7.591590625" y1="33.626590625" x2="7.62" y2="33.655" width="0.762" layer="16"/>
 <wire x1="7.62" y1="17.78" x2="5.715" y2="17.78" width="0.762" layer="16"/>
 <via x="5.715" y="17.78" extent="1-16" drill="0.35"/>
-<wire x1="5.715" y1="17.78" x2="5.08" y2="17.78" width="0.762" layer="1"/>
-<wire x1="5.08" y1="17.78" x2="3.81" y2="17.78" width="0.762" layer="1"/>
-<wire x1="5.08" y1="17.78" x2="5.08" y2="17.78" width="0.762" layer="1"/>
+<wire x1="5.715" y1="17.78" x2="3.81" y2="17.78" width="0.762" layer="1"/>
 </signal>
 <signal name="PA9">
@@
 <wire x1="1.27" y1="41.17" x2="7.515" y2="41.17" width="1.27" layer="1"/>
 <wire x1="7.515" y1="41.17" x2="7.62" y2="41.275" width="1.27" layer="1"/>
-<contactref element="SJ2" pad="2"/>
-<wire x1="6.35" y1="22.86" x2="4.5452" y2="24.6648" width="0.762" layer="16"/>
-<wire x1="4.5452" y1="24.6648" x2="4.5452" y2="37.8948" width="0.762" layer="16"/>
+<contactref element="VBAT" pad="2"/>
+<wire x1="7.62" y1="22.86" x2="4.5452" y2="25.9348" width="0.762" layer="16"/>
+<wire x1="4.5452" y1="25.9348" x2="4.5452" y2="37.8948" width="0.762" layer="16"/>
 <wire x1="4.5452" y1="37.8948" x2="1.27" y2="41.17" width="0.762" layer="16"/>
 </signal>
@@
 <signal name="N$1">
 <contactref element="A1" pad="4.1"/>
-<contactref element="SJ2" pad="1"/>
-<wire x1="8.89" y1="22.86" x2="8.89" y2="27.94" width="0.762" layer="16"/>
+<contactref element="VBAT" pad="1"/>
+<wire x1="10.16" y1="26.67" x2="8.89" y2="27.94" width="0.762" layer="16"/>
+<wire x1="10.16" y1="26.67" x2="10.16" y2="22.86" width="0.762" layer="16"/>
 </signal>
 <signal name="N$2">
 <contactref element="A1" pad="4.4"/>
 <wire x1="16.51" y1="23.495" x2="16.51" y2="27.94" width="0.762" layer="16"/>
-<contactref element="SJ3" pad="1"/>
+<contactref element="5V" pad="1"/>
 <wire x1="10.16" y1="17.78" x2="10.795" y2="17.78" width="0.762" layer="16"/>
 <wire x1="10.795" y1="17.78" x2="16.51" y2="23.495" width="0.762" layer="16"/>
