File: Nucleo Pepi board/schematic.brd (EAGLE design)
At the start: 64.8 x 67.3 mm, 11 parts, among them J1 1X2-3.5MM

Commit message: update pc
Parts:
- removed 5V: (no value), jumper:SJW
Connections:
- net N$2: no longer 5V.1
- net PA10: now also SERVO1.10; no longer SERVO1.7
- net PA11: now also SERVO2.10; no longer SERVO1.10
- net PA12: now also SERVO1.7; no longer SERVO1.13
- net PA2: now also ADC_DAC.1; no longer ADC.4
- net PA3: now also ADC.4; no longer ADC.1
- net PA4: now also ADC.1; no longer ADC_DAC.10
- net PA5: now also ADC_DAC.10; no longer ADC_DAC.7
- net PA6: now also ADC_DAC.7; no longer ADC_DAC.4
- net PA7: now also ADC_DAC.4; no longer ADC_DAC.1
- net PA8: now also SERVO2.13; no longer SERVO1.1
- net PA9: now also SERVO1.13; no longer SERVO1.4
- net PB0: now also SERVO1.4; no longer SERVO2.1
- net PB1: now also SERVO1.1; no longer SERVO2.4
- net PB3: now also SERVO2.1; no longer SERVO2.7
- net PB4: now also SERVO2.4; no longer SERVO2.10
- net PB5: now also SERVO2.7; no longer SERVO2.13
- net VCC: no longer 5V.2
Routing:
- net GND: track 169.6 -> 6.79 mm
- net N$2: track 13.2 -> 0.00 mm
- net PA11: track 33.4 -> 24.2 mm, vias 1 -> 0
- net PB0: track 18.9 -> 9.94 mm, vias 1 -> 0
- net PA2: track 38.2 -> 29.3 mm
- net VCC: track 107.0 -> 100.2 mm, vias 1 -> 0
- net PA4: track 20.0 -> 26.5 mm
- net PA3: track 21.0 -> 26.5 mm
- net 3V3: track 20.5 -> 25.0 mm
- net PA9: track 13.8 -> 9.94 mm, vias 1 -> 0
- net PA1: track 22.8 -> 26.5 mm
- net PA0: track 22.8 -> 26.5 mm
- net PB3: track 35.6 -> 32.2 mm
- net PB7: track 21.5 -> 24.4 mm, vias 1 -> 0
- net PA12: track 12.1 -> 9.94 mm
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- added copper zone on layer 1, net GND
- added copper zone on layer 16, net GND
Other:
- board text added: "Pepi Board Ver 1.4"

Commit message: v1.4
Routing:
- net PA11: track 24.2 -> 13.8 mm
- net PA2: track 29.3 -> 22.4 mm
- net PB3: track 32.2 -> 28.5 mm
- net PA3: track 26.5 -> 22.8 mm
- net PA0: track 26.5 -> 22.8 mm
- net PA4: track 26.5 -> 22.9 mm
- net PA1: track 26.5 -> 22.9 mm
- net PB4: track 17.2 -> 13.8 mm
- net PB5: track 17.2 -> 14.0 mm
- net VCC: track 100.2 -> 103.3 mm
- net PB6: track 24.4 -> 21.4 mm
- net PA8: track 16.8 -> 14.0 mm
- net PB7: track 24.4 -> 21.8 mm
- net GND: vias 0 -> 6
Other:
- board text removed: "Pepi Board Ver 1.3"
