File: Nucleo Pepi board/schematic.sch (EAGLE design)
At the start: 11 parts, among them J1 1X2-3.5MM

Commit message: update pc
Parts:
- removed 5V: (no value), jumper:SJW
Connections:
- net N$2: no longer 5V.1
- net PA10: now also SERVO1.10; no longer SERVO1.7
- net PA11: now also SERVO2.10; no longer SERVO1.10
- net PA12: now also SERVO1.7; no longer SERVO1.13
- net PA2: now also ADC_DAC.1; no longer ADC.4
- net PA3: now also ADC.4; no longer ADC.1
- net PA4: now also ADC.1; no longer ADC_DAC.10
- net PA5: now also ADC_DAC.10; no longer ADC_DAC.7
- net PA6: now also ADC_DAC.7; no longer ADC_DAC.4
- net PA7: now also ADC_DAC.4; no longer ADC_DAC.1
- net PA8: now also SERVO2.13; no longer SERVO1.1
- net PA9: now also SERVO1.13; no longer SERVO1.4
- net PB0: now also SERVO1.4; no longer SERVO2.1
- net PB1: now also SERVO1.1; no longer SERVO2.4
- net PB3: now also SERVO2.1; no longer SERVO2.7
- net PB4: now also SERVO2.4; no longer SERVO2.10
- net PB5: now also SERVO2.7; no longer SERVO2.13
- net VCC: no longer 5V.2
